File: ORION_VV_driver_v3.kicad_pcb (KiCad board)
At the start: 4 copper layers, 52.4 x 123.1 mm, 119 parts, among them J11 Conn_01x02, J12 Conn_01x05, J13 Conn_01x05, J14 Conn_01x03, J15 Conn_01x02, J2 Conn_01x04, J3 Conn_01x04, J4 Conn_01x06, J5 Conn_01x07, J6 Conn_01x07, Q1 IRF8721PBF-1, Q10 IRF8721PBF-1, Q11 IRF8721PBF-1, Q12 IRF8721PBF-1, Q2 IRF8721PBF-1, Q3 IRF8721PBF-1, Q4 IRF8721PBF-1, Q5 IRF8721PBF-1, Q6 IRF8721PBF-1, Q7 IRF8721PBF-1, Q8 IRF8721PBF-1, Q9 IRF8721PBF-1, SW1 SW_Push, SW2 SW_Push, SW3 SW_Push, SW4 SW_Push, SW5 SW_Push, U2 L78L15_SOT89, U3 MAX3051, U5 INA199, U6 INA199, Y1 Resonator

Commit message: ビアうち
Routing:
- net GND: vias 84 -> 88
Changed lines of the file:
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@@
   (via (at 114.5 61.5) (size 1) (drill 0.8) (layers "F.Cu" "B.Cu") (free) (net 77))
   (via (at 119 133) (size 0.8) (drill 0.4) (layers "F.Cu" "B.Cu") (free) (net 77))
+  (via (at 94.5 147.5) (size 1) (drill 0.8) (layers "F.Cu" "B.Cu") (free) (net 77))
   (via (at 107.5 112) (size 0.8) (drill 0.4) (layers "F.Cu" "B.Cu") (free) (net 77))
   (via (at 122 75) (size 0.8) (drill 0.4) (layers "F.Cu" "B.Cu") (free) (net 77))
@@
   (via (at 108.5 139.5) (size 0.8) (drill 0.4) (layers "F.Cu" "B.Cu") (free) (net 77))
   (via (at 112 135.5) (size 1) (drill 0.8) (layers "F.Cu" "B.Cu") (free) (net 77))
+  (via (at 92.5 54.5) (size 1) (drill 0.8) (layers "F.Cu" "B.Cu") (free) (net 77))
   (via (at 105.9 107.6) (size 0.8) (drill 0.4) (layers "F.Cu" "B.Cu") (net 77))
   (via (at 93 65) (size 1) (drill 0.8) (layers "F.Cu" "B.Cu") (free) (net 77))
   (via (at 113 136.5) (size 1) (drill 0.8) (layers "F.Cu" "B.Cu") (free) (net 77))
+  (via (at 94.5 52.5) (size 1) (drill 0.8) (layers "F.Cu" "B.Cu") (free) (net 77))
   (via (at 117.5 133) (size 0.8) (drill 0.4) (layers "F.Cu" "B.Cu") (free) (net 77))
   (via (at 117 138.5) (size 1) (drill 0.8) (layers "F.Cu" "B.Cu") (free) (net 77))
@@
   (via (at 119.5 64.5) (size 1) (drill 0.8) (layers "F.Cu" "B.Cu") (free) (net 77))
   (via (at 109.5 99.2755) (size 0.8) (drill 0.4) (layers "F.Cu" "B.Cu") (net 77))
+  (via (at 92 145.5) (size 1) (drill 0.8) (layers "F.Cu" "B.Cu") (free) (net 77))
   (via (at 121.5 66.5) (size 1) (drill 0.8) (layers "F.Cu" "B.Cu") (free) (net 77))
   (via (at 123 123) (size 0.8) (drill 0.4) (layers "F.Cu" "B.Cu") (free) (net 77))

Commit message: hoge
Parts:
- moved C25 0.71 mm to (123.5, 64.5)
- moved C27 0.71 mm to (121.5, 62.5)
- moved C29 0.71 mm to (117.5, 58.5)
- moved C30 0.71 mm to (119.5, 60.5)
- moved C36 0.50 mm to (124.5, 68.0)
- moved C37 0.50 mm to (124.5, 70.5)
Routing:
- net /M1_VL: track 58.2 -> 55.9 mm
- net +12V: track 169.5 -> 167.5 mm
- net /M1_WL: track 52.5 -> 50.5 mm
- net /M1_UL: track 55.3 -> 53.3 mm
- net /M1_WH: track 65.8 -> 63.8 mm
- net /M1_VH: track 70.7 -> 68.7 mm
- net /M1_UH: track 71.9 -> 69.9 mm
- net /M0_W: track 27.6 -> 26.8 mm, vias 13 -> 25
- net Net-(GD1-Pad13): track 24.8 -> 25.6 mm
- net GND: vias 88 -> 200
- net /M1_W: vias 13 -> 21
- net /M1_V: vias 10 -> 20
- net /M1_U: vias 13 -> 24
- net /M1_CSL: vias 33 -> 155
- net /M0_V: vias 10 -> 18
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